File: final_project/board/hoop_detector.brd (EAGLE design)
At the start: 89 x 55 mm, 59 parts

Commit message: board
Parts:
- removed PAD59: (no value), wirepad:1,6/0,9
- added PAD15, PAD60, PAD65, PAD66, PAD67, PAD68, PAD69: (no value), wirepad:1,6/0,9
- moved PAD44 77.7 mm to (66.0, 26.7)
- moved PAD29 52.2 mm to (87.6, 16.5)
- moved PAD2 52.1 mm to (66.0, 31.8)
- moved PAD16 49.9 mm to (94.0, 59.7)
- moved PAD32 49.9 mm to (94.0, 57.1)
- moved PAD33 49.9 mm to (94.0, 54.6)
- moved PAD34 49.9 mm to (94.0, 52.1)
- moved PAD35 49.9 mm to (94.0, 49.5)
- moved PAD36 49.9 mm to (94.0, 47.0)
- moved PAD37 49.9 mm to (94.0, 44.5)
- moved PAD38 49.9 mm to (94.0, 41.9)
- moved PAD39 49.9 mm to (94.0, 39.4)
- moved PAD40 49.9 mm to (94.0, 36.8)
- moved PAD41 49.9 mm to (94.0, 34.3)
- moved PAD42 49.9 mm to (94.0, 29.2)
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Connections:
- net N$12: now also PAD67.1, PAD68.1, PAD69.1; no longer PAD44.1
- net N$13: now also PAD65.1, PAD66.1
- net N$16: now also PAD15.1, PAD60.1
- net N$27: now also PAD2.1; no longer PAD59.1
- net N$29: now also PAD44.1; no longer PAD2.1
Routing:
- net N$13: track 7.71 -> 49.5 mm
- net N$12: track 7.85 -> 35.6 mm
- net N$16: track 0.00 -> 10.2 mm
- net N$29: track 7.83 -> 6.35 mm
- net N$27: track 7.70 -> 6.35 mm
- net N$21: track 7.70 -> 6.43 mm, vias 0 -> 1
- net N$4: track 7.71 -> 6.44 mm, vias 0 -> 1
- net N$9: track 7.85 -> 6.58 mm, vias 0 -> 1
- net N$3: track 7.85 -> 6.58 mm, vias 0 -> 1
- net N$15: track 7.85 -> 6.58 mm, vias 0 -> 1
- net N$28: track 7.62 -> 6.35 mm
- net N$26: track 7.83 -> 6.56 mm, vias 0 -> 1
- net N$25: track 7.62 -> 6.35 mm
- net N$22: track 7.62 -> 6.35 mm
- net N$20: track 7.83 -> 6.56 mm, vias 0 -> 1
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
Commit message: finish board pcb
Parts:
- added PAD59, PAD61, PAD62, PAD63: (no value), wirepad:1,6/0,9
- added R1: (no value), resistor:0204/7
- added SP1: KSS1201, buzzer:KSS1201
- added SW1: (no value), special:EDG-02
- moved PAD48 75.8 mm to (141.0, 40.6)
- moved PAD46 45.7 mm to (67.3, 11.4)
- moved PAD47 43.6 mm to (72.4, 11.4)
- moved PAD49 21.6 mm to (66.0, 27.9)
- moved PAD56 21.6 mm to (66.0, 50.8)
- moved PAD55 14.0 mm to (66.0, 48.3)
- moved PAD50 11.4 mm to (66.0, 35.6)
- moved PAD54 8.89 mm to (66.0, 45.7)
- moved PAD51 6.35 mm to (66.0, 38.1)
- moved PAD60 6.35 mm to (66.0, 53.3)
- moved PAD53 3.81 mm to (66.0, 43.2)
- moved PAD10 1.27 mm to (68.6, 45.7)
- moved PAD11 1.27 mm to (68.6, 48.3)
- moved PAD12 1.27 mm to (68.6, 50.8)
- moved PAD19 1.27 mm to (91.4, 50.8)
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Connections:
- removed net N$16: PAD15.1, PAD60.1, U$1.D13
- removed net N$19: PAD12.1, PAD48.1, U$1.A0
- removed net N$20: PAD11.1, PAD49.1, U$1.A1
- removed net N$21: PAD10.1, PAD50.1, U$1.A2
- removed net N$22: PAD51.1, PAD9.1, U$1.A3
- removed net N$24: PAD53.1, PAD7.1, U$1.A5
- removed net N$25: PAD54.1, PAD6.1, U$1.A6
- new net N$36: SP1.-
- new net N$38: PAD46.1, R1.2
- new net N$39: PAD14.1, PAD61.1, U$1.3.3V
- new net N$40: PAD13.1, PAD60.1, U$1.AREF
- new net N$41: PAD12.1, PAD56.1, U$1.A0
- new net N$42: PAD10.1, PAD54.1, U$1.A2
- new net N$43: PAD53.1, PAD9.1, U$1.A3
- new net N$45: PAD51.1, PAD7.1, U$1.A5
- new net N$46: PAD50.1, PAD6.1, U$1.A6
- new net N$47: PAD11.1, PAD55.1, U$1.A1
- new net N$48: PAD15.1, PAD62.1, U$1.D13
- net N$12: now also PAD47.1
- net N$13: now also SW1.3
- net N$17: now also PAD59.1, SW1.2; no longer PAD14.1, PAD46.1, U$1.3.3V
- net N$18: now also SP1.+, SW1.4; no longer PAD13.1, PAD47.1, U$1.AREF
- net N$26: now also PAD63.1, R1.1; no longer PAD55.1
- net N$28: now also PAD49.1; no longer PAD56.1
Routing:
- net N$12: track 35.6 -> 160.4 mm
- net N$47: track 0.00 -> 105.1 mm, vias 0 -> 1
- net N$13: track 49.5 -> 97.4 mm
- net N$18: track 6.43 -> 30.0 mm, vias 1 -> 0
- net N$16: track 10.2 -> 0.00 mm
- net N$26: track 6.56 -> 16.5 mm
- net N$38: track 0.00 -> 8.13 mm
- net N$17: track 6.56 -> 0.00 mm, vias 1 -> 0
- net N$20: track 6.56 -> 0.00 mm, vias 1 -> 0
- net N$39: track 0.00 -> 6.44 mm, vias 0 -> 1
- net N$24: track 6.43 -> 0.00 mm, vias 1 -> 0
- net N$21: track 6.43 -> 0.00 mm, vias 1 -> 0
- net N$42: track 0.00 -> 6.36 mm, vias 0 -> 1
- net N$45: track 0.00 -> 6.36 mm, vias 0 -> 1
- net N$40: track 0.00 -> 6.36 mm, vias 0 -> 1
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Other:
- board text added: "ARDUINO"
- board text added: "LED"
- board text added: "SPEAKER"
- board text added: "SWITCH"
