File: final_project/board/hoop_detector.sch (EAGLE design)
At the start: 59 parts

Commit message: board
Parts:
- removed PAD59: (no value), wirepad:1,6/0,9
- added PAD15, PAD60, PAD65, PAD66, PAD67, PAD68, PAD69: (no value), wirepad:1,6/0,9
Connections:
- net N$12: now also PAD67.P, PAD68.P, PAD69.P; no longer PAD44.P
- net N$13: now also PAD65.P, PAD66.P
- net N$16: now also PAD15.P, PAD60.P
- net N$27: now also PAD2.P; no longer PAD59.P
- net N$29: now also PAD44.P; no longer PAD2.P
Other:
- moved on the sheet: PAD1, PAD10, PAD11, PAD12, PAD13, PAD14, PAD16, PAD17, PAD18, PAD19, PAD2, PAD20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

Commit message: finish board pcb
Parts:
- added PAD59, PAD61, PAD62, PAD63: (no value), wirepad:1,6/0,9
- added R1: (no value), resistor:R-US_0204/7
- added SP1: KSS1201, buzzer:KSS1201
- added SW1: (no value), special:SW_DIP-2
Connections:
- removed net N$16: PAD15.P, PAD60.P, U$1.D13
- removed net N$19: PAD12.P, PAD48.P, U$1.A0
- removed net N$20: PAD11.P, PAD49.P, U$1.A1
- removed net N$21: PAD10.P, PAD50.P, U$1.A2
- removed net N$22: PAD51.P, PAD9.P, U$1.A3
- removed net N$24: PAD53.P, PAD7.P, U$1.A5
- removed net N$25: PAD54.P, PAD6.P, U$1.A6
- new net N$36: SP1.2
- new net N$38: PAD46.P, R1.2
- new net N$39: PAD14.P, PAD61.P, U$1.3.3V
- new net N$40: PAD13.P, PAD60.P, U$1.AREF
- new net N$41: PAD12.P, PAD56.P, U$1.A0
- new net N$42: PAD10.P, PAD54.P, U$1.A2
- new net N$43: PAD53.P, PAD9.P, U$1.A3
- new net N$45: PAD51.P, PAD7.P, U$1.A5
- new net N$46: PAD50.P, PAD6.P, U$1.A6
- new net N$47: PAD11.P, PAD55.P, U$1.A1
- new net N$48: PAD15.P, PAD62.P, U$1.D13
- net N$12: now also PAD47.P
- net N$13: now also SW1.3
- net N$17: now also PAD59.P, SW1.2; no longer PAD14.P, PAD46.P, U$1.3.3V
- net N$18: now also SP1.1, SW1.4; no longer PAD13.P, PAD47.P, U$1.AREF
- net N$26: now also PAD63.P, R1.1; no longer PAD55.P
- net N$28: now also PAD49.P; no longer PAD56.P
Other:
- moved on the sheet: PAD15, PAD44, PAD46, PAD47, PAD48, PAD49, PAD50, PAD51, PAD52, PAD53, PAD54, PAD55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
